File: chainable_halfdigit_controller.sch (KiCad schematic (older format))
At the start: 3 parts, among them J1 USB_OTG, U1 NRF24L01, U2 arduino_nano

Commit message: Made custom ST-USB-013A footprint for mini usb connector
Parts:
- J1: footprint Connectors_USB:USB_Micro-B_Molex-105017-0001 -> lib_fp:ST-USB-013A
Changed lines of the file:
@@
 EESchema Schematic File Version 2
 LIBS:arduino
-LIBS:nRF24L01+
 LIBS:NRF24L01
 LIBS:power
@@
 F 0 "J1" H 7100 3750 50  0000 L CNN
 F 1 "USB_OTG" H 7100 3650 50  0000 L CNN
-F 2 "Connectors_USB:USB_Micro-B_Molex-105017-0001" H 7450 3250 50  0001 C CNN
+F 2 "lib_fp:ST-USB-013A" H 7450 3250 50  0001 C CNN
 F 3 "" H 7450 3250 50  0001 C CNN
 	1    7300 3300

Commit message: Added bluetooth connection, board outline and mounting holes
Parts:
- added J2: Conn_01x06, Socket_Strips:Socket_Strip_Angled_1x06_Pitch2.54mm, symbol Conn_01x06
Connections:
- net +3V3: now also J2.2 (Pin_2)
- net GND: now also J2.3 (Pin_3)
- net BL_TXD: now reaches U2.22 (D4)
- net BL_TXD: now also J2.4 (Pin_4)
- net BL_RXD: now reaches U2.23 (#D5)
- net BL_RXD: now also J2.5 (Pin_5)
- net IRQ: no longer names the net of U1.8 (IRQ)
- no-connect marks 24 -> 25
Changed lines of the file:
@@
 NoConn ~ 4050 4100
 NoConn ~ 4050 4000
-NoConn ~ 4050 3900
-NoConn ~ 4050 3800
 NoConn ~ 4050 3550
 NoConn ~ 4050 3250
@@
 Text GLabel 6300 2600 2    60   Input ~ 0
 CSN
-Text GLabel 6300 2750 2    60   Input ~ 0
-IRQ
 Text GLabel 5250 2900 0    60   Input ~ 0
 SCK
@@
 Text GLabel 5250 2600 0    60   Input ~ 0
 MISO
+NoConn ~ 2650 4700
+$Comp
+L Conn_01x06 J2
+U 1 1 5A1DE956
+P 6750 4850
+F 0 "J2" H 6750 5150 50  0000 C CNN
+F 1 "Conn_01x06" H 6750 4450 50  0000 C CNN
+F 2 "Socket_Strips:Socket_Strip_Angled_1x06_Pitch2.54mm" H 6750 4850 50  0001 C CNN
+F 3 "" H 6750 4850 50  0001 C CNN
+	1    6750 4850
+	1    0    0    -1
+$EndComp
+Text GLabel 6200 5150 0    60   Input ~ 0
+BL_RXD
+Text GLabel 6200 5000 0    60   Input ~ 0
+BL_TXD
+Text GLabel 6200 4700 0    60   Input ~ 0
+3V3
+Text GLabel 6200 4850 0    60   Input ~ 0
+GND
+Text GLabel 4250 3900 2    60   Input ~ 0
+BL_TXD
+Text GLabel 4250 3800 2    60   Input ~ 0
+BL_RXD
+NoConn ~ 6550 4650
+NoConn ~ 6550 5150
+NoConn ~ 6150 2750
 Wire Wire Line
 	7050 3850 7400 3850
 Wire Wire Line
-	7200 3850 7200 3700
+	7200 3700 7200 4100
 Wire Wire Line
 	7300 3850 7300 3700
@@
 Connection ~ 7300 3850
 Wire Wire Line
-	3350 5200 3350 5050
-Wire Wire Line
 	3200 2150 3200 2350
 Wire Wire Line
@@
 Connection ~ 3500 2250
 Wire Wire Line
-	4200 2850 4050 2850
-Wire Wire Line
 	4050 2950 4200 2950
 Wire Wire Line
@@
 Wire Wire Line
 	5750 3250 5750 3100
-NoConn ~ 2650 4700
 Connection ~ 7050 3850
 Connection ~ 3650 2250
 Wire Wire Line
-	6300 2750 6150 2750
+	6550 4850 6200 4850
+Wire Wire Line
+	6550 4750 6350 4750
+Wire Wire Line
+	6350 4750 6350 4700
+Wire Wire Line
+	6350 4700 6200 4700
+Wire Wire Line
+	6550 4950 6350 4950
+Wire Wire Line
+	6350 4950 6350 5000
+Wire Wire Line
+	6350 5000 6200 5000
+Wire Wire Line
+	6550 5050 6400 5050
+Wire Wire Line
+	6400 5050 6400 5150
+Wire Wire Line
+	6400 5150 6200 5150
+Wire Wire Line
+	4250 3800 4050 3800
+Wire Wire Line
+	4250 3900 4050 3900
+Wire Wire Line
+	4050 2850 4200 2850
+Wire Wire Line
+	3350 5200 3350 5050
+$Comp
+L PWR_FLAG #FLG05
+U 1 1 5A1DFFDB
+P 7200 4100
+F 0 "#FLG05" H 7200 4175 50  0001 C CNN
+F 1 "PWR_FLAG" H 7200 4250 50  0000 C CNN
+F 2 "" H 7200 4100 50  0001 C CNN
+F 3 "" H 7200 4100 50  0001 C CNN
+	1    7200 4100
+	-1   0    0    1
+$EndComp
 $EndSCHEMATC

Commit message: Added banana jack and pin header for power switch
Parts:
- added J3, J4: Conn_01x01, Connectors:Banana_Jack_1Pin, symbol Conn_01x01
- added SW1: SW_SPST, Pin_Headers:Pin_Header_Straight_1x02_Pitch2.54mm, symbol SW_SPST
Connections:
- net +5V: now also J3.1 (Pin_1), SW1.1 (A); no longer U2.15 (Vin)
- new net 5V: J4.1 (Pin_1), SW1.2 (B), U2.15 (Vin)
Changed lines of the file:
@@
 NoConn ~ 7600 3400
 NoConn ~ 7600 3500
-Text GLabel 8000 3100 2    60   Input ~ 0
+Text GLabel 9750 3100 2    60   Input ~ 0
 5V
 Text GLabel 7400 3850 3    60   Input ~ 0
@@
 L PWR_FLAG #FLG01
 U 1 1 5A1B46DB
-P 7650 2950
-F 0 "#FLG01" H 7650 3025 50  0001 C CNN
-F 1 "PWR_FLAG" H 7650 3100 50  0000 C CNN
-F 2 "" H 7650 2950 50  0001 C CNN
-F 3 "" H 7650 2950 50  0001 C CNN
-	1    7650 2950
+P 7800 2950
+F 0 "#FLG01" H 7800 3025 50  0001 C CNN
+F 1 "PWR_FLAG" H 7800 3100 50  0000 C CNN
+F 2 "" H 7800 2950 50  0001 C CNN
+F 3 "" H 7800 2950 50  0001 C CNN
+	1    7800 2950
 	1    0    0    -1
 $EndComp
@@
 L +5V #PWR03
 U 1 1 5A1B47CF
-P 7950 2950
-F 0 "#PWR03" H 7950 2800 50  0001 C CNN
-F 1 "+5V" H 7950 3090 50  0000 C CNN
-F 2 "" H 7950 2950 50  0001 C CNN
-F 3 "" H 7950 2950 50  0001 C CNN
-	1    7950 2950
+P 8100 2950
+F 0 "#PWR03" H 8100 2800 50  0001 C CNN
+F 1 "+5V" H 8100 3090 50  0000 C CNN
+F 2 "" H 8100 2950 50  0001 C CNN
+F 3 "" H 8100 2950 50  0001 C CNN
+	1    8100 2950
 	1    0    0    -1
 $EndComp
@@
 	7300 3850 7300 3700
 Wire Wire Line
-	7600 3100 8000 3100
-Wire Wire Line
-	7650 2950 7650 3100
-Connection ~ 7650 3100
-Wire Wire Line
-	7950 2950 7950 3100
-Connection ~ 7950 3100
+	7600 3100 8400 3100
+Wire Wire Line
+	7800 2950 7800 3100
+Connection ~ 7800 3100
+Wire Wire Line
+	8100 2950 8100 3100
+Connection ~ 8100 3100
 Connection ~ 7200 3850
 Connection ~ 7300 3850
@@
 	3200 2150 3200 2350
 Wire Wire Line
-	3500 2350 3500 2150
+	3500 2150 3500 2350
 Wire Wire Line
 	3650 2250 3500 2250
@@
 	-1   0    0    1
 $EndComp
+$Comp
+L SW_SPST SW1
+U 1 1 5A22D5DE
+P 8850 2650
+F 0 "SW1" H 8850 2775 50  0000 C CNN
+F 1 "SW_SPST" H 8850 2550 50  0000 C CNN
+F 2 "Pin_Headers:Pin_Header_Straight_1x02_Pitch2.54mm" H 8850 2650 50  0001 C CNN
+F 3 "" H 8850 2650 50  0001 C CNN
+	1    8850 2650
+	1    0    0    -1
+$EndComp
+$Comp
+L Conn_01x01 J3
+U 1 1 5A22E23B
+P 8600 3100
+F 0 "J3" H 8600 3200 50  0000 C CNN
+F 1 "Conn_01x01" H 8600 3000 50  0000 C CNN
+F 2 "Connectors:Banana_Jack_1Pin" H 8600 3100 50  0001 C CNN
+F 3 "" H 8600 3100 50  0001 C CNN
+	1    8600 3100
+	1    0    0    -1
+$EndComp
+$Comp
+L Conn_01x01 J4
+U 1 1 5A22E27D
+P 9000 3100
+F 0 "J4" H 9000 3200 50  0000 C CNN
+F 1 "Conn_01x01" H 9000 3000 50  0000 C CNN
+F 2 "Connectors:Banana_Jack_1Pin" H 9000 3100 50  0001 C CNN
+F 3 "" H 9000 3100 50  0001 C CNN
+	1    9000 3100
+	-1   0    0    1
+$EndComp
+Wire Wire Line
+	9200 3100 9750 3100
+Wire Wire Line
+	8400 3100 8400 2650
+Wire Wire Line
+	8400 2650 8650 2650
+Wire Wire Line
+	9200 3100 9200 2650
+Wire Wire Line
+	9200 2650 9050 2650
+$Comp
+L PWR_FLAG #FLG06
+U 1 1 5A22E915
+P 2950 2250
+F 0 "#FLG06" H 2950 2325 50  0001 C CNN
+F 1 "PWR_FLAG" H 2950 2400 50  0000 C CNN
+F 2 "" H 2950 2250 50  0001 C CNN
+F 3 "" H 2950 2250 50  0001 C CNN
+	1    2950 2250
+	1    0    0    -1
+$EndComp
+Wire Wire Line
+	3200 2350 2950 2350
+Wire Wire Line
+	2950 2350 2950 2250
 $EndSCHEMATC

Commit message: Fixed DRC errors
Changed lines of the file:
@@
 Wire Wire Line
 	2950 2350 2950 2250
+$Comp
+L PWR_FLAG #FLG07
+U 1 1 5A2B29A5
+P 4050 2800
+F 0 "#FLG07" H 4050 2875 50  0001 C CNN
+F 1 "PWR_FLAG" H 4050 2950 50  0000 C CNN
+F 2 "" H 4050 2800 50  0001 C CNN
+F 3 "" H 4050 2800 50  0001 C CNN
+	1    4050 2800
+	1    0    0    -1
+$EndComp
+Wire Wire Line
+	4050 2850 4050 2800
 $EndSCHEMATC
